File: ESP32 S2 MCU.kicad_sch (KiCad schematic)
At the start: 22 parts, among them U11 ESP32-S2, X3 40MHz

Commit message: Created Production Files and Added Rendering. Just need to add silkscreen of pinout
Parts:
- X3: LCSC C669071 -> C717687
Other:
- company: (none) -> Niko Smith
- title: (none) -> VehicleVCU
Changed lines of the file:
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@@
 (kicad_sch (version 20230121) (generator eeschema)
   (paper "A4")
+  (title_block
+    (title "VehicleVCU")
+    (date "2023-06-26")
+    (rev "V2.0")
+    (company "Niko Smith")
+  )
   (junction (at 181.61 29.21) (diameter 0) (color 0 0 0 0)
   )
@@
       (effects (font (size 1.27 1.27)) hide)
     )
-    (property "LCSC" "C669071" (at 36.83 100.33 0)
-      (effects (font (size 1.27 1.27)) hide)
-    )
+    (property "LCSC" "C717687" (at 36.83 100.33 0)
+      (effects (font (size 1.27 1.27)) hide)
+    )
