File: VehicleVCU_PCB.kicad_pcb (KiCad board)
At the start: 4 copper layers, 60 x 85 mm, 86 parts, among them J1 USB_B, J2 ATM13-08, Q1 BC847BS, Q2 SSM3J328, SW1 Button 1, SW2 Button 1, SW3 Button 1, U1 USBLC6-2SC6, U10 AMS1117-5, U2 ESP32-S2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

Commit message: Final Commit. Created ibom
Other:
- board text added: "1: GLV+ 2: CAN3L 3: CAN2L 4: CAN1L 5: CAN1H 6: CAN2H 7: CAN3H 8: GND"
